Commit message: adding neck pan tilt controller and modernize xacro load_yaml

File: config/a200_0876.ros2_control.xacro (robot description, xacro)
@@ -2,5 +2,5 @@
 <robot xmlns:xacro="http://www.ros.org/wiki/xacro">
     <xacro:macro name="a200_0876_ros2_control" params="name initial_positions_file">
-        <xacro:property name="initial_positions" value="${load_yaml(initial_positions_file)['initial_positions']}"/>
+        <xacro:property name="initial_positions" value="${xacro.load_yaml(initial_positions_file)['initial_positions']}"/>
         <ros2_control name="${name}" type="system">
             <hardware>

File: config/a200_0876.urdf.xacro (robot description, xacro)
@@ -5,6 +5,9 @@
     <!-- Import a200_0876 urdf file -->
     <xacro:include filename="$(find husky_description)/urdf/robot.urdf.xacro" />
-    <!-- Import control_xacro -->
+    <!-- Import mock control xacro for arms + grippers -->
     <xacro:include filename="a200_0876.ros2_control.xacro" />
     <xacro:a200_0876_ros2_control name="FakeSystem" initial_positions_file="$(arg initial_positions_file)"/>
+    <!-- Import neck pan/tilt control (dynamixel_hardware in dummy mode by default) -->
+    <xacro:include filename="$(find husky_description)/urdf/control/neck_ros2_control.xacro" />
+    <xacro:neck_ros2_control name="neck_dynamixels"/>
 </robot>
